File: udb-s.kicad_sch (KiCad schematic)
At the start: 10 parts, among them J1 TYPE-C-31-M-12, J2 78171-0004, U1 TPD4E05U06DQAR

Commit message: added kikit panel assembly
Parts:
- D1: LCSC (none) -> C502546; LCSC Part Number C502546 -> (none)
- F1: LCSC (none) -> C2833485; LCSC Part Number C2833485 -> (none)
- FB1: LCSC (none) -> C1017; LCSC Part Number C1017 -> (none)
- J1: JLCPCB_CORRECTION (none) -> 0; -5; 0; LCSC (none) -> C165948; LCSC Part Number C165948 -> (none)
- J2: JLCPCB_CORRECTION (none) -> 0; 0; 0; LCSC (none) -> C528030; LCSC Part Number C588524 -> (none)
- R1, R2: LCSC (none) -> C138073
- U1: JLCPCB_CORRECTION (none) -> 0; 0; 270; LCSC (none) -> C2836386; LCSC Part Number C2836386 -> (none)
Changed lines of the file:
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@@
       (effects (font (size 1.27 1.27)) hide)
     )
-    (property "LCSC Part Number" "C2833485" (id 6) (at 241.3 44.45 0)
+    (property "LCSC" "C2833485" (id 6) (at 241.3 44.45 0)
       (effects (font (size 1.27 1.27)) hide)
     )
@@
       (effects (font (size 1.27 1.27)) hide)
     )
-    (property "LCSC Part Number" "C1017" (id 6) (at 122.555 103.505 0)
+    (property "LCSC" "C1017" (id 6) (at 122.555 103.505 0)
       (effects (font (size 1.27 1.27)) hide)
     )
@@
       (effects (font (size 1.27 1.27)) hide)
     )
-    (property "LCSC Part Number" "C165948" (id 6) (at 105.41 67.945 0)
+    (property "LCSC" "C165948" (id 6) (at 105.41 67.945 0)
+      (effects (font (size 1.27 1.27)) hide)
+    )
+    (property "JLCPCB_CORRECTION" "0; -5; 0" (id 7) (at 105.41 67.945 0)
       (effects (font (size 1.27 1.27)) hide)
     )
@@
       (effects (font (size 1.27 1.27)) hide)
     )
-    (property "LCSC Part Number" "C2836386" (id 9) (at 177.8 98.425 0)
+    (property "LCSC" "C2836386" (id 9) (at 177.8 98.425 0)
+      (effects (font (size 1.27 1.27)) hide)
+    )
+    (property "JLCPCB_CORRECTION" "0; 0; 270" (id 10) (at 177.8 98.425 0)
       (effects (font (size 1.27 1.27)) hide)
     )
@@
       (effects (font (size 1.27 1.27)) hide)
     )
-    (property "LCSC Part Number" "C588524" (id 6) (at 173.99 46.355 0)
+    (property "LCSC" "C528030" (id 6) (at 173.99 46.355 0)
+      (effects (font (size 1.27 1.27)) hide)
+    )
+    (property "JLCPCB_CORRECTION" "0; 0; 0" (id 7) (at 173.99 46.355 0)
       (effects (font (size 1.27 1.27)) hide)
     )
@@
       (effects (font (size 1.27 1.27)) hide)
     )
-    (property "LCSC Part Number" "C502546" (id 6) (at 228.6 50.8 0)
+    (property "LCSC" "C502546" (id 6) (at 228.6 50.8 0)
       (effects (font (size 1.27 1.27)) hide)
     )
@@
       (effects (font (size 1.27 1.27)) hide)
     )
+    (property "LCSC" "C138073" (id 4) (at 130.175 57.785 0)
+      (effects (font (size 1.27 1.27)) hide)
+    )
     (pin "1")
     (pin "2")
@@
       (effects (font (size 1.27 1.27)) hide)
     )
+    (property "LCSC" "C138073" (id 4) (at 130.175 60.325 0)
+      (effects (font (size 1.27 1.27)) hide)
+    )
